File: PCB/88-CCC Board 1/88-CCC Board 1.kicad_sch (KiCad schematic)
At the start: 38 parts, among them J11 To Board 2, J17 To Cyclops, P1 S100_MALE, Q1 2N3646, U12 74151, U13 7408, U14 7493, U15 7475, U16 7404, U21 7493, U22 7402, U23 7474, U24 74193, U25 7483, U26 7483, U27 7420, U28 7493, U31 7474, U32 7475, U33 7475, U34 7475, U35 7475, U36 7475, U37 7474, U38 74193, U41 74367, U42 7404, U43 7404, U44 74367, U45 74367, U46 74LS10, U47 7474, U48 7474

Commit message: Board 1 schematic updates
Connections:
- net +5V: now also U13.14 (VCC), U16.14 (VCC), U22.14 (VCC), U23.14 (VCC), U24.5 (UP), U27.14 (VCC), U31.14 (VCC), U37.14 (VCC), U38.15 (A), U38.5 (UP), U42.14 (VCC), U43.14 (VCC), U46.14 (VCC), U47.14 (VCC), U48.14 (VCC)
- net GND: now also U13.7 (GND), U16.7 (GND), U22.7 (GND), U23.7 (GND), U27.7 (GND), U31.7 (GND), U37.7 (GND), U42.7 (GND), U43.7 (GND), U46.7 (GND), U47.7 (GND), U48.7 (GND)
- net at U32.8 (~{Q3}): now also J17.15 (Pin_15), U41.10 (I4)
- now unconnected: U32.9 (Q3)
- no-connect marks 23 -> 56
Other:
- moved on the sheet: C1, J11, J17, P1, Q1, R1, R2, R3, R4, U12, U13A, U13B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

Commit message: Board 1 Schematics Update
Parts:
- added C10, C11: 47uF, Capacitor_THT:C_Axial_L12.0mm_D9.5mm_P20.00mm_Horizontal, symbol Device:C_Polarized
- added C2, C3, C4, C5, C6, C7, C8, C9: 0.1uF, Capacitor_THT:C_Disc_D7.5mm_W5.0mm_P5.00mm, symbol Device:C_Small
- C1: footprint (none) -> Capacitor_THT:C_Disc_D7.5mm_W5.0mm_P5.00mm
- U12, U25: footprint (none) -> Package_DIP:DIP-16_W7.62mm
- U14, U21, U28: footprint Package_DIP:DIP-10_W7.62mm -> Package_DIP:DIP-14_W7.62mm
- U31: footprint Package_DIP:DIP-14_W7.62mm_SMDSocket_SmallPads -> Package_DIP:DIP-14_W7.62mm
Connections:
- net +5V: now also C10.1, C11.1, C2.1, C3.1, C4.1, C5.1, C6.1, C7.1, C8.1, C9.1
- net GND: now also C10.2, C11.2, C2.2, C3.2, C4.2, C5.2, C6.2, C7.2, C8.2, C9.2

Commit message: Schematic updates
Parts:
- added U18: L7805, Package_TO_SOT_THT:TO-220-3_Horizontal_TabDown, symbol Regulator_Linear:L7805
- J11, J17: footprint Connector_IDC:IDC-Header_2x08_P2.54mm_Vertical -> Package_DIP:DIP-16_W7.62mm
Connections:
- net +5V: now also U18.3 (OUT); no longer C10.1
- net GND: now also P1.50 (0_V2), U18.2 (GND)
- net +8V: now reaches P1.1 (+8_V)
- net +8V: now also C10.1, P1.51 (+8_V), U18.1 (IN)
- net -17V renamed -16V
Other:
- moved on the sheet: C10, C11

Commit message: Board 1 PCB
Parts:
- U27: footprint Package_DIP:DIP-12_W7.62mm -> Package_DIP:DIP-14_W7.62mm
Changed lines of the file:
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@@
 			)
 		)
-		(property "Footprint" "Package_DIP:DIP-12_W7.62mm"
+		(property "Footprint" "Package_DIP:DIP-14_W7.62mm"
 			(at 222.25 212.09 0)
 			(effects
@@
 			)
 		)
-		(property "Footprint" "Package_DIP:DIP-12_W7.62mm"
+		(property "Footprint" "Package_DIP:DIP-14_W7.62mm"
 			(at 245.11 271.78 0)
 			(effects
@@
 			)
 		)
-		(property "Footprint" "Package_DIP:DIP-12_W7.62mm"
+		(property "Footprint" "Package_DIP:DIP-14_W7.62mm"
 			(at 111.76 36.83 0)
 			(effects

Commit message: Board 1 PCB
Parts:
- C1, C2, C3, C4, C5, C6, C7, C8, C9: footprint Capacitor_THT:C_Disc_D7.5mm_W5.0mm_P5.00mm -> Capacitor_THT:C_Disc_D7.5mm_W5.0mm_P7.50mm
- C10, C11: footprint Capacitor_THT:C_Axial_L12.0mm_D9.5mm_P20.00mm_Horizontal -> Capacitor_THT:C_Axial_L17.0mm_D7.0mm_P25.00mm_Horizontal
- Q1: footprint Package_TO_SOT_THT:TO-39-3 -> Package_TO_SOT_THT:TO-92
- R1, R2, R3, R4: footprint footprints:R1206 -> Resistor_THT:R_Axial_DIN0207_L6.3mm_D2.5mm_P10.16mm_Horizontal; LCSC Part C1469 -> (none)
Changed lines of the file:
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@@
 			)
 		)
-		(property "Footprint" "footprints:R1206"
+		(property "Footprint" "Resistor_THT:R_Axial_DIN0207_L6.3mm_D2.5mm_P10.16mm_Horizontal"
 			(at 291.084 129.794 90)
 			(effects
@@
 			)
 		)
-		(property "LCSC Part" "C1469"
+		(property "LCSC Part" ""
 			(at 290.83 130.81 0)
 			(effects
@@
 			)
 		)
-		(property "Footprint" "Capacitor_THT:C_Axial_L12.0mm_D9.5mm_P20.00mm_Horizontal"
+		(property "Footprint" "Capacitor_THT:C_Axial_L17.0mm_D7.0mm_P25.00mm_Horizontal"
 			(at 540.7152 41.91 0)
 			(effects
@@
 			)
 		)
-		(property "Footprint" "Capacitor_THT:C_Disc_D7.5mm_W5.0mm_P5.00mm"
+		(property "Footprint" "Capacitor_THT:C_Disc_D7.5mm_W5.0mm_P7.50mm"
 			(at 58.42 73.66 0)
 			(effects
@@
 			)
 		)
-		(property "Footprint" "Capacitor_THT:C_Disc_D7.5mm_W5.0mm_P5.00mm"
+		(property "Footprint" "Capacitor_THT:C_Disc_D7.5mm_W5.0mm_P7.50mm"
 			(at 38.1 73.66 0)
 			(effects
@@
 			)
 		)
-		(property "Footprint" "Capacitor_THT:C_Axial_L12.0mm_D9.5mm_P20.00mm_Horizontal"
+		(property "Footprint" "Capacitor_THT:C_Axial_L17.0mm_D7.0mm_P25.00mm_Horizontal"
 			(at 507.6952 41.91 0)
 			(effects
@@
 			)
 		)
-		(property "Footprint" "footprints:R1206"
+		(property "Footprint" "Resistor_THT:R_Axial_DIN0207_L6.3mm_D2.5mm_P10.16mm_Horizontal"
 			(at 350.266 94.234 90)
 			(effects
@@
 			)
 		)
-		(property "LCSC Part" "C1469"
+		(property "LCSC Part" ""
 			(at 349.25 93.98 0)
 			(effects
@@
 			)
 		)
-		(property "Footprint" "Capacitor_THT:C_Disc_D7.5mm_W5.0mm_P5.00mm"
+		(property "Footprint" "Capacitor_THT:C_Disc_D7.5mm_W5.0mm_P7.50mm"
 			(at 349.25 111.76 0)
 			(effects
@@
 			)
 		)
-		(property "Footprint" "footprints:R1206"
+		(property "Footprint" "Resistor_THT:R_Axial_DIN0207_L6.3mm_D2.5mm_P10.16mm_Horizontal"
 			(at 484.124 87.884 90)
 			(effects
@@
 			)
 		)
-		(property "LCSC Part" "C1469"
+		(property "LCSC Part" ""
 			(at 483.87 88.9 0)
 			(effects
@@
 			)
 		)
-		(property "Footprint" "Package_TO_SOT_THT:TO-39-3"
+		(property "Footprint" "Package_TO_SOT_THT:TO-92"
 			(at 505.46 90.805 0)
 			(effects
@@
 			)
 		)
-		(property "Footprint" "Capacitor_THT:C_Disc_D7.5mm_W5.0mm_P5.00mm"
+		(property "Footprint" "Capacitor_THT:C_Disc_D7.5mm_W5.0mm_P7.50mm"
 			(at 99.06 73.66 0)
 			(effects
@@
 			)
 		)
-		(property "Footprint" "footprints:R1206"
+		(property "Footprint" "Resistor_THT:R_Axial_DIN0207_L6.3mm_D2.5mm_P10.16mm_Horizontal"
 			(at 291.084 119.634 90)
 			(effects
@@
 			)
 		)
-		(property "LCSC Part" "C1469"
+		(property "LCSC Part" ""
 			(at 290.83 120.65 0)
 			(effects
@@
 			)
 		)
-		(property "Footprint" "Capacitor_THT:C_Disc_D7.5mm_W5.0mm_P5.00mm"
+		(property "Footprint" "Capacitor_THT:C_Disc_D7.5mm_W5.0mm_P7.50mm"
 			(at 78.74 73.66 0)
 			(effects
@@
 			)
 		)
-		(property "Footprint" "Capacitor_THT:C_Disc_D7.5mm_W5.0mm_P5.00mm"
+		(property "Footprint" "Capacitor_THT:C_Disc_D7.5mm_W5.0mm_P7.50mm"
 			(at 68.58 73.66 0)
 			(effects
@@
 			)
 		)
-		(property "Footprint" "Capacitor_THT:C_Disc_D7.5mm_W5.0mm_P5.00mm"
+		(property "Footprint" "Capacitor_THT:C_Disc_D7.5mm_W5.0mm_P7.50mm"
 			(at 88.9 73.66 0)
 			(effects
@@
 			)
 		)
-		(property "Footprint" "Capacitor_THT:C_Disc_D7.5mm_W5.0mm_P5.00mm"
+		(property "Footprint" "Capacitor_THT:C_Disc_D7.5mm_W5.0mm_P7.50mm"
 			(at 27.94 73.66 0)
 			(effects
@@
 			)
 		)
-		(property "Footprint" "Capacitor_THT:C_Disc_D7.5mm_W5.0mm_P5.00mm"
+		(property "Footprint" "Capacitor_THT:C_Disc_D7.5mm_W5.0mm_P7.50mm"
 			(at 48.26 73.66 0)
 			(effects
