File: PCB/88-CCC Board 1/88-CCC Board 1.kicad_pcb (KiCad board)
At the start: 6 copper layers, 254 x 134.6 mm, 206 parts, among them J1 to WDI, J2 44-pin IDE, J3 Serial, J4 40-pin IDE, J5 EXT PWR, J6 Jumper to enable buzzer, P1 S100_MALE, P7 5V Reg, Q1 2N2222AU, SW1 SW_DIP_x07, U1 Z80CPU, U10 74HCT240, U101 74HCT138, U102 74LS123, U103 74LS123, U104 74HCT00, U11 74HCT374, U13 74HCT244, U14 74F138, U15 74HCT138, U16 74F138, U17 7438, U18 7438, U19 7438, U2 28C256, U20 7438, U21 74LS123, U22 74LS123, U23 74HCT165, U24 74HCT374, U25 74HCT164, U26 74F163, U27 74HCT393, U28 74HCT74, U29 74HCT138, U3 CY62256NLL-55ZXIT, U30 74HCT74, U31 74HCT374, U32 74HCT244, U33 74HCT244, U34 74HCT374, U35 74HCT374, U36 75107, U37 75110, U38 74HCT04, U39 74F04, U4 2681, U40 74F00, U41 74F08, U42 74F08, U43 74HCT32, U44 74HCT04, U45 74HCT14, U46 74HCT163, U47 74HCT02, U48 7905, U5 MAX232A, U50 3.3V LDO Reg, U6 74F74, U7 74F74, U8 74HCT374, U9 74LS244

Commit message: Cleared PCB
Parts:
- removed BZ1: Buzzer, Buzzer_Beeper:Buzzer_12x9.5RM7.6
- removed C1, C10, C11, C13, C15, C16, C17, C18, C24, C25, C26, C27, C28, C29, C30, C31, C32, C36, C37, C38, C40, C41, C42, C44, C45, C46, C47, C48, C49, C50, C51, C52, C53, C54, C55, C56, C57, C58, C59, C6, C60, C61, C62, C63, C64, C65, C66, C67, C68, C69, C74, C75, C77, C78, C8, C9: 0.1uF, footprints:C0603
- removed C12, C14, C71, C73: 10uF, footprints:CAP-SMD_BD4.0-L4.3-W4.3-FD
- removed C19, C7: 47uF, footprints:CAP-SMD_BD6.3-L6.6-W6.6-FD
- removed C2, C3, C4: 1.0uF, footprints:C0603
- removed C20: 22uF, footprints:C0603
- removed C21, C22, C23: 470pF, footprints:C0603
- removed C33, C34, C35, C39: 47pF, footprints:C0603
- removed C43: 22pF, footprints:C0603
- removed C5: 4.7uF, footprints:CAP-SMD_BD4.0-L4.3-W4.3-LS5.3-FD
- removed C70, C72: 33uF, footprints:CAP-SMD_BD6.3-L6.6-W6.6-FD
- removed C76: .33uF, footprints:C0603
- removed D1: 1N4148W T4, footprints:SOD-123_L2.8-W1.8-LS3.7-RD
- removed D3: BAT41, Diode_THT:D_DO-35_SOD27_P7.62mm_Horizontal
- removed J1: to WDI, Connector_IDC:IDC-Header_2x17_P2.54mm_Vertical
- removed J2: 44-pin IDE, footprints:SAMTEC-SQT-122-01-X-D-RA
- removed J3: Serial, Connector_PinHeader_2.54mm:PinHeader_1x05_P2.54mm_Vertical
- removed J4: 40-pin IDE, Connector_IDC:IDC-Header_2x20_P2.54mm_Vertical
- removed J5: EXT PWR, Connector_PinHeader_2.54mm:PinHeader_1x03_P2.54mm_Vertical
- removed J6: Jumper to enable buzzer, Connector_PinHeader_2.54mm:PinHeader_2x01_P2.54mm_Vertical
- removed LED1, LED2, LED3, LED4: YELLOW, footprints:LED0805-R-RD
- removed LED11, LED12, LED13, LED6, LED9: RED, footprints:LED0805-R-RD
- removed LED5, LED7, LED8: GREEN, footprints:LED0805-R-RD
- removed OSC1: 3.6864MHz, footprints:OSC-SMD_4P-L7.0-W5.0-BL-2
- removed OSC2: 27MHz, footprints:OSC-SMD_4P-L7.0-W5.0-BL-2
- removed OSC3: 22.5792MHz, footprints:OSC-SMD_4P-L7.0-W5.0-BL-2
- removed P7: 5V Reg, Connector_PinHeader_2.54mm:PinHeader_1x05_P2.54mm_Vertical
- removed Q1: 2N2222AU, footprints:SOT-89-3_L4.5-W2.4-P1.50-LS4.0-BR
- removed R1, R2, R3, R4: 270, footprints:R0603
- removed R10: 100, Resistor_THT:R_Axial_DIN0207_L6.3mm_D2.5mm_P10.16mm_Horizontal
- removed R11, R12, R13: 100K, footprints:R1206
- removed R14, R30: 270K, footprints:R1206
- removed R15, R23, R24, R25, R26, R27, R28, R29: 4.7K, footprints:R1206
- removed R18: 47K, footprints:R1206
- removed R22, R31, R50, R6, R9: 360, footprints:R0603
- removed R32: 2.2K, footprints:R1206
- removed R33, R37, R39, R41, R46, R47, R52: 1K, footprints:R1206
- removed R34, R35, R36: 15K, footprints:R1206
- removed R38, R53: 1.5K, footprints:R1206
- removed R40: 470, footprints:R1206
- removed R44, R45: 33, footprints:R1206
- removed R48: 5.6K, footprints:R1206
- removed R49: 10K, footprints:R1206
- removed R5, R7, R8: 160, footprints:R0603
- removed R51: 100, footprints:R1206
- removed RP1: 761-5-R220/330, Package_DIP:DIP-16_W7.62mm
- removed RP2: 4x100Ω, Resistor_THT:R_Array_SIP8
- removed SW1: SW_DIP_x07, Package_DIP:DIP-14_W7.62mm
- removed U1: Z80CPU, Package_DIP:DIP-40_W15.24mm
- removed U10: 74HCT240, footprints:TSSOP-20_L6.5-W4.4-P0.65-LS6.5-BL
- removed U101, U15, U29: 74HCT138, footprints:TSSOP-16_L5.0-W4.4-P0.65-LS6.4-BL
- removed U102, U103, U21, U22: 74LS123, footprints:SOIC-16_L9.9-W3.9-P1.27-LS6.0-BL
- removed U104: 74HCT00, footprints:TSSOP-14_L5.0-W4.4-P0.65-LS6.4-BL
- removed U11, U24, U31, U34, U35, U8: 74HCT374, footprints:SOP-20_L12.6-W5.3-P1.27-LS7.8-BL
- removed U13, U32, U33: 74HCT244, footprints:TSSOP-20_L6.5-W4.4-P0.65-LS6.4-BL
- removed U14, U16: 74F138, Package_DIP:DIP-16_W7.62mm
- removed U17, U18, U19, U20: 7438, Package_DIP:DIP-14_W7.62mm
- removed U2: 28C256, Package_DIP:DIP-28_W15.24mm
- removed U23: 74HCT165, footprints:SOIC-16_L9.9-W3.9-P1.27-LS6.0-BL
- removed U25: 74HCT164, footprints:TSSOP-14_L5.0-W4.4-P0.65-LS6.4-BL
- removed U26: 74F163, footprints:SOIC-16_L9.9-W3.9-P1.27-LS6.0-BL
- removed U27: 74HCT393, footprints:SO-14_L8.7-W3.9-P1.27-LS6.0-BL
- removed U28, U30: 74HCT74, footprints:SO-14_L8.9-W3.9-P1.27-LS6.0-BL
- removed U3: CY62256NLL-55ZXIT, footprints:TSOP-28_L11.8-W8.0-P0.55-LS13.4-B_CYPRESS
- removed U36: 75107, Package_DIP:DIP-14_W7.62mm
- removed U37: 75110, Package_DIP:DIP-14_W7.62mm
- removed U38, U44: 74HCT04, footprints:TSSOP-14_L5.0-W4.4-P0.65-LS6.4-BL
- removed U39: 74F04, footprints:SOIC-14_L8.7-W3.9-P1.27-LS6.0-BL
- removed U4: 2681, Package_DIP:DIP-24_W10.16mm
- removed U40: 74F00, footprints:SOIC-14_L8.7-W3.9-P1.27-LS6.0-BL
- removed U41, U42: 74F08, footprints:SSOP-14_L6.2-W5.3-P0.65-LS7.8-BL-1
- removed U43: 74HCT32, footprints:TSSOP-14_L5.0-W4.4-P0.65-LS6.4-BL
- removed U45: 74HCT14, footprints:TSSOP-14_L5.0-W4.4-P0.65-LS6.4-BL
- removed U46: 74HCT163, footprints:SOIC-16_L9.9-W3.9-P1.27-LS6.0-BL
- removed U47: 74HCT02, footprints:SOIC-14_L8.7-W3.9-P1.27-LS6.0-BL
- removed U48: 7905, footprints:TO-252-2_L6.6-W6.1-P4.57-LS10.1-BR-CW
- removed U5: MAX232A, Package_DIP:DIP-16_W7.62mm
- removed U50: 3.3V LDO Reg, footprints:SOIC-8_L5.0-W4.0-P1.27-LS6.0-BL
- removed U6, U7: 74F74, footprints:SOIC-14_L8.7-W3.9-P1.27-LS6.0-BL
- removed U9: 74LS244, footprints:SOP-20_L12.6-W5.3-P1.27-LS7.8-BL
Routing:
- net +5V: track 1692.8 -> 0.00 mm, vias 2 -> 0
- net GND: track 182.2 -> 0.00 mm
- net Net-(J5-Pin_2): track 100.4 -> 0.00 mm, vias 1 -> 0
- net Net-(J5-Pin_1): track 60.6 -> 0.00 mm
- net -5V: track 39.5 -> 0.00 mm
- net Net-(C39-Pad1): track 37.1 -> 0.00 mm
- net Net-(C39-Pad2): track 36.8 -> 0.00 mm
- net Net-(OSC3-EOH): track 22.7 -> 0.00 mm
- net Net-(U103B-RCext): track 19.8 -> 0.00 mm
- net Net-(D1-A): track 18.3 -> 0.00 mm
- net Net-(U103B-Cext): track 11.5 -> 0.00 mm
- net Net-(C33-Pad1): track 11.2 -> 0.00 mm
- net Net-(U102B-RCext): track 10.4 -> 0.00 mm
- net Net-(U103A-RCext): track 9.43 -> 0.00 mm
- net Net-(U21A-RCext): track 8.09 -> 0.00 mm
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- removed copper zone on B.Cu, net GND
- removed copper zone on F.Cu, net GND
Other:
- board text removed: "+8V"
- board text removed: "-16V"
- board text removed: "Buzzer Enable"
- board text removed: "Design: Mike Arnold / PCB: Aron Hoekstra"
- board text removed: "External IDE"
- board text removed: "External Power"
- board text removed: "FAULT"
- board text removed: "FLUSH"
- board text removed: "GND"
- board text removed: "HD0"
- board text removed: "HD1"
- board text removed: "HD2"
- board text removed: "HD3"
- board text removed: "IDE"
- board text removed: "READ"
- board text removed: "REV 1"
- board text removed: "ROM"
- board text removed: "RxA"
- board text removed: "RxB"
- board text removed: "SEEK"
- board text removed: "SEL"
- board text removed: "Serial/Debug"
- board text removed: "TxA"
- board text removed: "TxB"
- board text removed: "W2I - Cromemco WDI to IDE adapter"
- board text removed: "WDI"
- board text removed: "WRITE"

Commit message: Board 1 PCB
Parts:
- added C1: 150pf, Capacitor_THT:C_Disc_D7.5mm_W5.0mm_P5.00mm, F.Cu at (-105.1, 13.3)
- added C10: 47uF, Capacitor_THT:C_Axial_L12.0mm_D9.5mm_P20.00mm_Horizontal, F.Cu at (-40.8, 7.95)
- added C11: 47uF, Capacitor_THT:C_Axial_L12.0mm_D9.5mm_P20.00mm_Horizontal, F.Cu at (-20.0, 67.5)
- added C2: 0.1uF, Capacitor_THT:C_Disc_D7.5mm_W5.0mm_P5.00mm, F.Cu at (-105.1, 19.8)
- added C3: 0.1uF, Capacitor_THT:C_Disc_D7.5mm_W5.0mm_P5.00mm, F.Cu at (-105.1, 26.4)
- added C4: 0.1uF, Capacitor_THT:C_Disc_D7.5mm_W5.0mm_P5.00mm, F.Cu at (-96.0, 13.3)
- added C5: 0.1uF, Capacitor_THT:C_Disc_D7.5mm_W5.0mm_P5.00mm, F.Cu at (-96.0, 19.8)
- added C6: 0.1uF, Capacitor_THT:C_Disc_D7.5mm_W5.0mm_P5.00mm, F.Cu at (-96.0, 26.4)
- added C7: 0.1uF, Capacitor_THT:C_Disc_D7.5mm_W5.0mm_P5.00mm, F.Cu at (-87.0, 13.3)
- added C8: 0.1uF, Capacitor_THT:C_Disc_D7.5mm_W5.0mm_P5.00mm, F.Cu at (-87.0, 19.8)
- added C9: 0.1uF, Capacitor_THT:C_Disc_D7.5mm_W5.0mm_P5.00mm, F.Cu at (255.0, 45.0)
- added G***: LOGO, Dazzler:bd1-Overlay-bottom, F.Cu at (82.0, 56.5)
- added J11: To Board 2, Package_DIP:DIP-16_W7.62mm, F.Cu at (228.7, 50.1)
- added J17: To Cyclops, Package_DIP:DIP-16_W7.62mm, F.Cu at (55.9, 50.0)
- added Q1: 2N3646, Package_TO_SOT_THT:TO-39-3, F.Cu at (-71.2, 15.5)
- added R1: 560, footprints:R1206, F.Cu at (-77.0, 11.6)
- added R2: 1.5K, footprints:R1206, F.Cu at (-77.0, 14.9)
- added R3: 1K, footprints:R1206, F.Cu at (-77.0, 18.3)
- added R4: 4.7K, footprints:R1206, F.Cu at (-77.0, 21.6)
- added U12: 74151, Package_DIP:DIP-16_W7.62mm, F.Cu at (198.6, 50.1)
- added U13: 7408, Package_DIP:DIP-14_W7.62mm, F.Cu at (170.0, 50.1)
- added U14: 7493, Package_DIP:DIP-14_W7.62mm, F.Cu at (142.5, 50.1)
- added U15: 7475, Package_DIP:DIP-16_W7.62mm, F.Cu at (112.4, 50.1)
- added U16: 7404, Package_DIP:DIP-14_W7.62mm, F.Cu at (84.8, 50.1)
- added U18: L7805, Package_TO_SOT_THT:TO-220-3_Horizontal_TabDown, F.Cu at (27.7, 62.8)
- added U21: 7493, Package_DIP:DIP-14_W7.62mm, F.Cu at (230.0, 76.0)
- added U22: 7402, Package_DIP:DIP-14_W7.62mm, F.Cu at (200.0, 76.0)
- added U23: 7474, Package_DIP:DIP-14_W7.62mm, F.Cu at (170.0, 76.0)
- added U24: 74193, Package_DIP:DIP-16_W7.62mm, F.Cu at (141.2, 76.0)
- added U25: 7483, Package_DIP:DIP-16_W7.62mm, F.Cu at (112.4, 76.0)
- added U26: 7483, Package_DIP:DIP-16_W7.62mm, F.Cu at (83.6, 76.0)
- added U27: 7420, Package_DIP:DIP-14_W7.62mm, F.Cu at (57.3, 76.0)
- added U28: 7493, Package_DIP:DIP-14_W7.62mm, F.Cu at (29.8, 76.0)
- added U31: 7474, Package_DIP:DIP-14_W7.62mm, F.Cu at (230.0, 101.0)
- added U32: 7475, Package_DIP:DIP-16_W7.62mm, F.Cu at (198.7, 101.0)
- added U33: 7475, Package_DIP:DIP-16_W7.62mm, F.Cu at (168.7, 101.0)
- added U34: 7475, Package_DIP:DIP-16_W7.62mm, F.Cu at (141.2, 101.0)
- added U35: 7475, Package_DIP:DIP-16_W7.62mm, F.Cu at (112.4, 101.0)
- added U36: 7475, Package_DIP:DIP-16_W7.62mm, F.Cu at (83.6, 101.0)
- added U37: 7474, Package_DIP:DIP-14_W7.62mm, F.Cu at (57.3, 101.0)
- added U38: 74193, Package_DIP:DIP-16_W7.62mm, F.Cu at (28.6, 101.0)
- added U41: 74367, Package_DIP:DIP-16_W7.62mm, F.Cu at (228.6, 127.0)
- added U42: 7404, Package_DIP:DIP-14_W7.62mm, F.Cu at (199.8, 127.0)
- added U43: 7404, Package_DIP:DIP-14_W7.62mm, F.Cu at (169.9, 127.0)
- added U44: 74367, Package_DIP:DIP-16_W7.62mm, F.Cu at (141.0, 127.0)
- added U45: 74367, Package_DIP:DIP-16_W7.62mm, F.Cu at (112.3, 127.0)
- added U46: 74LS10, Package_DIP:DIP-14_W7.62mm, F.Cu at (84.8, 127.0)
- added U47: 7474, Package_DIP:DIP-14_W7.62mm, F.Cu at (57.4, 127.0)
- added U48: 7474, Package_DIP:DIP-14_W7.62mm, F.Cu at (29.6, 127.0)
Connections:
- P1 pad 1: Net-(J5-Pin_1) -> +8V
- P1 pad 2: unconnected-(P1-+16_V-Pad2) -> +16V
- P1 pad 26: unconnected-(P1-pHDLA-Pad26) -> PHLDA
- P1 pad 32: unconnected-(P1-A15-Pad32) -> A15
- P1 pad 33: unconnected-(P1-A12-Pad33) -> A12
- P1 pad 34: unconnected-(P1-A9-Pad34) -> A9
- P1 pad 35: unconnected-(P1-DO1-Pad35) -> D01
- P1 pad 36: unconnected-(P1-DO0-Pad36) -> D00
- P1 pad 37: unconnected-(P1-A10-Pad37) -> A10
- P1 pad 38: unconnected-(P1-DO4-Pad38) -> D04
- P1 pad 39: unconnected-(P1-DO5-Pad39) -> D05
- P1 pad 40: unconnected-(P1-DO6-Pad40) -> D06
- P1 pad 41: unconnected-(P1-D12-Pad41) -> D12
- P1 pad 42: unconnected-(P1-D13-Pad42) -> D13
- P1 pad 43: unconnected-(P1-D17-Pad43) -> D17
- P1 pad 51: unconnected-(P1-+8_V-Pad51) -> +8V
- P1 pad 52: Net-(J5-Pin_2) -> -16V
- P1 pad 73: unconnected-(P1-INT*-Pad73) -> PINT
- P1 pad 75: /S100_RESET_P75 -> PRESET
- P1 pad 76: unconnected-(P1-pSYNC-Pad76) -> PSYNC
- P1 pad 83: unconnected-(P1-A7-Pad83) -> A7
- P1 pad 84: unconnected-(P1-A8-Pad84) -> A8
- P1 pad 85: unconnected-(P1-A13-Pad85) -> A13
- P1 pad 86: unconnected-(P1-A14-Pad86) -> A14
- P1 pad 87: unconnected-(P1-A11-Pad87) -> A11
- P1 pad 88: unconnected-(P1-DO2-Pad88) -> D02
- P1 pad 89: unconnected-(P1-DO3-Pad89) -> D03
- P1 pad 90: unconnected-(P1-DO7-Pad90) -> D07
- P1 pad 93: unconnected-(P1-DI6-Pad93) -> D16
- P1 pad 94: unconnected-(P1-DI1-Pad94) -> D11
- P1 pad 95: unconnected-(P1-DI0-Pad95) -> D10
Other:
- copper layers 6 -> 2
- board text added: "1"
- board text added: "2"
- board text added: "3"
- board text added: "4"
- board text added: "8 7 6 5 4 3 2 1"
- board text added: "CROMEMCO 88 CCC BOARD 1"
- board text added: "REPRODUCTION 2026 ARON HOEKSTRA"
- board text added: "TO CYCLOPS"

Commit message: Board 1 PCB
Parts:
- C1, C2, C3, C4, C5, C6, C7, C8, C9: footprint Capacitor_THT:C_Disc_D7.5mm_W5.0mm_P5.00mm -> Capacitor_THT:C_Disc_D7.5mm_W5.0mm_P7.50mm
- C10, C11: footprint Capacitor_THT:C_Axial_L12.0mm_D9.5mm_P20.00mm_Horizontal -> Capacitor_THT:C_Axial_L17.0mm_D7.0mm_P25.00mm_Horizontal
- Q1: footprint Package_TO_SOT_THT:TO-39-3 -> Package_TO_SOT_THT:TO-92
- R1, R2, R3, R4: footprint footprints:R1206 -> Resistor_THT:R_Axial_DIN0207_L6.3mm_D2.5mm_P10.16mm_Horizontal
- moved R3 247.0 mm to (136.7, 142.0), turned to 180 degrees
- moved Q1 227.0 mm to (117.5, 141.6)
- moved C1 214.0 mm to (80.8, 119.4), turned to -90 degrees
- moved R4 181.7 mm to (76.7, 118.4), turned to -90 degrees
- moved R2 167.4 mm to (88.9, 37.0), turned to 180 degrees
- moved R1 143.4 mm to (59.5, 55.3)
- moved C2 122.1 mm to (-4.75, 89.5)
- moved C3 122.1 mm to (-4.75, 96.0)
- moved C10 100.5 mm to (23.2, 85.4), turned to 90 degrees
- moved C11 71.5 mm to (23.5, 124.2), turned to 90 degrees
- moved C9 17.2 mm to (242.5, 33.2)
- moved C6 16.7 mm to (-85.2, 39.1)
Routing:
- net +5V: track 0.00 -> 1187.9 mm, vias 0 -> 12
- net GND: track 0.00 -> 1106.0 mm, vias 0 -> 16
Other:
- board text added: "1.5K"
- board text added: "1K"
- board text added: "2N3646"
- board text added: "560"
- board text added: "7402"
- board text added: "7404"
- board text added: "7408"
- board text added: "74151"
- board text added: "74193"
- board text added: "7420"
- board text added: "74367"
- board text added: "7474"
- board text added: "7475"
- board text added: "7483"
- board text added: "7493"
- board text added: "74LS10"
- board text added: "TO BOARD 2"

Commit message: Board 1 PCB
Parts:
- moved C7 350.6 mm to (253.7, 96.2)
- moved C6 349.0 mm to (253.7, 122.2)
- moved C8 344.5 mm to (253.7, 71.0)
- moved C5 176.7 mm to (79.2, 42.5), turned to -90 degrees
- moved C4 157.2 mm to (51.1, 68.5), turned to -90 degrees
- moved C2 50.6 mm to (23.8, 131.2)
- moved C3 30.1 mm to (24.6, 89.3)
- moved C9 16.5 mm to (253.7, 45.3)
- moved U18 2.49 mm to (27.6, 60.3)
Routing:
- net -16V: track 0.00 -> 115.9 mm, vias 0 -> 1
- net +16V: track 0.00 -> 108.7 mm
- net +5V: track 1187.9 -> 1264.3 mm, vias 12 -> 13
- net GND: track 1106.0 -> 1144.3 mm

Commit message: Reproduction PCBs Final
Parts:
- moved C2 7.92 mm to (30.1, 136.0)
- moved R4 0.70 mm to (76.0, 118.4)
- moved C1 0.45 mm to (80.3, 119.4)
Routing:
- net Net-(J11-Pin_12): track 0.00 -> 264.8 mm, vias 0 -> 4
- net Net-(J11-Pin_3): track 0.00 -> 255.9 mm, vias 0 -> 4
- net Net-(J17-Pin_15): track 0.00 -> 250.5 mm, vias 0 -> 5
- net Net-(U31A-~{Q}): track 0.00 -> 250.2 mm, vias 0 -> 3
- net Net-(J17-Pin_13): track 0.00 -> 245.1 mm, vias 0 -> 4
- net Net-(J11-Pin_5): track 0.00 -> 240.0 mm, vias 0 -> 4
- net Net-(J17-Pin_14): track 0.00 -> 239.5 mm, vias 0 -> 5
- net Net-(J17-Pin_12): track 0.00 -> 235.2 mm, vias 0 -> 6
- net Net-(J11-Pin_15): track 0.00 -> 230.3 mm, vias 0 -> 2
- net Net-(U12-I1): track 0.00 -> 212.2 mm, vias 0 -> 2
- net Net-(U41-OEa): track 0.00 -> 211.8 mm, vias 0 -> 2
- net Net-(J11-Pin_7): track 0.00 -> 203.3 mm, vias 0 -> 1
- net Net-(U41-I5): track 0.00 -> 202.5 mm, vias 0 -> 1
- net Net-(J11-Pin_9): track 0.00 -> 201.1 mm, vias 0 -> 1
- net Net-(U23A-~{Q}): track 0.00 -> 188.6 mm, vias 0 -> 4
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