File: PCB/88-CCC Board 2/88-CCC Board 2.kicad_sch (KiCad schematic)
At the start: 12 parts, among them P1 S100_MALE, U18 L7805

Commit message: Board 2 Schematics
Parts:
- added J11: To Board 1, Package_DIP:DIP-16_W7.62mm, symbol Connector_Generic:Conn_02x08_Counter_Clockwise
- added J35: Port Select, Package_DIP:DIP-18_W7.62mm_LongPads, symbol Connector_Generic:Conn_02x09_Counter_Clockwise
- added U12, U13: 7493, Package_DIP:DIP-14_W7.62mm, symbol 74xx:74LS93
- added U14: 7430, Package_DIP:DIP-10_W7.62mm, symbol 74xx:74LS30
- added U15, U25: 7430, symbol 74xx:74LS30
- added U16, U17, U26, U27, U38: 7474, Package_DIP:DIP-14_W7.62mm, symbol 74xx:74LS74
- added U21: 74HC164, Package_DIP:DIP-14_W7.62mm, symbol 74xx:74HC164
- added U22, U23, U32, U33: 7475, Package_DIP:DIP-16_W7.62mm, symbol 74xx:74LS75
- added U24, U36: 7402, Package_DIP:DIP-14_W7.62mm, symbol 74xx:7402
- added U28, U37, U48: 7400, Package_DIP:DIP-14_W7.62mm, symbol 74xx:7400
- added U31, U41, U47: 7405, Package_DIP:DIP-14_W7.62mm, symbol 74xx:74LS05
- added U34: 7410, Package_DIP:DIP-14_W7.62mm, symbol 74xx:74LS10
- added U42, U43, U44: 74367, Package_DIP:DIP-16_W7.62mm, symbol 74xx:74LS367
- added U45, U46: 7404, Package_DIP:DIP-14_W7.62mm, symbol 74xx:74LS04

Commit message: Board 2 schematic updates
Parts:
- removed unit 3 of U36
- added R1: 1K, footprints:R1206, symbol Device:R_US
- added U1: 7402, Package_DIP:DIP-14_W7.62mm, symbol 74xx:7402
Connections:
- net +5V: now also U16.1 (~{R}), U16.10 (~{S}), U16.4 (~{S}), U17.10 (~{S}), U17.4 (~{S}), U26.1 (~{R}), U26.13 (~{R}), U26.4 (~{S}), U27.4 (~{S}), U38.10 (~{S}), U38.4 (~{S}), U44.16 (VCC), R1.1
- net PHLDA: now also U37.2
- net 02: now reaches P1.24 (PHI)
- net 02: now also U46.1
- net CLOCK: now reaches P1.49 (CLOCK)
- net CLOCK: now also U46.3
- net at U47.5: now also U38.12 (D), U47.13, U47.3
- net at U36.11: now also U1.10
- net at U36.12: now also U37.12
- net OUT: now reaches U36.13
- net at U46.2: now also U48.4, U48.5
- net at U37.4: now also U28.1, U28.6
- net at U37.5: now also U16.3 (C), U27.3 (C), U38.11 (C)
- net at U37.6: now also U38.1 (~{R})
- net IN: now reaches U34.1
- net IN: now also R1.2, U1.8, U1.9
- net at U34.12: now also U37.9
- net at U37.10: now also U37.11
- net at U37.8: now also U38.2 (D)
- net at U17.11 (C): now also U17.3 (C), U26.11 (C), U26.3 (C), U38.3 (C), U48.3
- net at U17.12 (D): now also U17.5 (Q)
- net at U17.13 (~{R}): now also U17.1 (~{R}), U17.2 (D), U37.13, U48.9
- net at U17.9 (Q): now also U37.1
- net at U13.9 (Q1): now also U23.6 (D2)
- net at J11.6 (Pin_6): now also U24.10
- net at U26.5 (Q): now also U26.12 (D)
- net at U26.6 (~{Q}): now also U36.5
- net at U28.4: now also U27.1 (~{R}), U27.2 (D), U28.3
- net at U28.5: now also U38.13 (~{R})
- net at U48.11: now also U48.10
- net at U48.12: now also U48.8
- net at U48.13: now also U37.3
- net at U28.2: now also U28.11
- net at U33.6 (D2): now also U12.9 (Q1)
- net at U36.4: now also U36.2, U36.3
- net at U36.6: now also U26.9 (Q)
- net at U26.8 (~{Q}): now also U16.2 (D)
- net at U44.4 (I2): now also U36.1
- net at U16.11 (C): now also U46.4
- net at U48.6: now also U48.2
- net at U31.11: now also U38.9 (Q)
- net A10: no longer names the net of P1.37 (A10)
- net A11: no longer names the net of P1.87 (A11)
- net A12: no longer names the net of P1.33 (A12)
- net A13: no longer names the net of P1.85 (A13)
- net A14: no longer names the net of P1.86 (A14)
- net A15: no longer names the net of P1.32 (A15)
- net A7: no longer names the net of P1.83 (A7)
- net A8: no longer names the net of P1.84 (A8)
- net A9: no longer names the net of P1.34 (A9)
- net D00: no longer names the net of P1.36 (DO0)
- net D01: no longer names the net of P1.35 (DO1)
- net D02: no longer names the net of P1.88 (DO2)
- net D03: no longer names the net of P1.89 (DO3)
- net D04: no longer names the net of P1.38 (DO4)
- net D05: no longer names the net of P1.39 (DO5)
- net D06: no longer names the net of P1.40 (DO6)
- net D07: no longer names the net of P1.90 (DO7)
- net D10: no longer names the net of P1.95 (DI0)
- net D11: no longer names the net of P1.94 (DI1)
- net D12: no longer names the net of P1.41 (D12)
- net D13: no longer names the net of P1.42 (D13)
- net D16: no longer names the net of P1.93 (DI6)
- net D17: no longer names the net of P1.43 (D17)
- net PINT: no longer names the net of P1.73 (INT*)
- net PRESET: no longer names the net of P1.75 (RESET*)
- net PSYNC: no longer names the net of P1.76 (pSYNC)
Other:
- moved on the sheet: J11, J35, U12, U13, U14A, U15A, U16A, U16B, U17A, U17B, U21, U22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

Commit message: Board 2 Schematics
Parts:
- removed J35: Port Select, Package_DIP:DIP-18_W7.62mm_LongPads, symbol Connector_Generic:Conn_02x09_Counter_Clockwise
- added R2: 560, footprints:R1206, symbol Device:R_US
- added SW1, SW2, SW3: SW_DPDT_x2, Package_DIP:DIP-6_W7.62mm, symbol Switch:SW_DPDT_x2
- added SW35: Port Select, Package_DIP:DIP-6_W7.62mm, symbol Switch:SW_DPDT_x2
Connections:
- net +5V: now also U12.5 (VCC), U13.5 (VCC), U14.14 (VCC), U15.14 (VCC), U16.13 (~{R}), U16.14 (VCC), U17.14 (VCC), U21.14 (VCC), U21.9 (~{MR}), U22.5 (VCC), U23.5 (VCC), U24.14 (VCC), U25.14 (VCC), U26.14 (VCC), U27.14 (VCC), U28.14 (VCC), U31.14 (VCC), U32.5 (VCC), U33.5 (VCC), U34.14 (VCC), U36.14 (VCC), U37.14 (VCC), U38.14 (VCC), U41.14 (VCC), U42.16 (VCC), U43.16 (VCC), U44.14 (I6), U44.2 (I1), U45.14 (VCC), U46.14 (VCC), U47.14 (VCC), U48.14 (VCC), R2.1
- net GND: now also J11.8 (Pin_8), U12.10 (GND), U13.10 (GND), U14.7 (GND), U15.7 (GND), U16.7 (GND), U17.7 (GND), U21.7 (GND), U22.12 (GND), U23.12 (GND), U24.7 (GND), U25.7 (GND), U26.7 (GND), U27.7 (GND), U28.7 (GND), U31.7 (GND), U32.12 (GND), U33.12 (GND), U34.7 (GND), U36.7 (GND), U37.7 (GND), U38.7 (GND), U41.7 (GND), U42.8 (GND), U43.8 (GND), U44.8 (GND), U45.7 (GND), U46.7 (GND), U47.7 (GND), U48.7 (GND)
- net SDSB: now reaches P1.18 (SDSB*)
- net SDSB: now also U47.12
- net CDSB: now reaches P1.19 (CDSB*)
- net CDSB: now also U47.4
- net ADSB: now reaches P1.22 (ADSB*)
- net ADSB: now also U47.10
- net DODSB: now reaches P1.23 (DODSB*)
- net DODSB: now also U47.6
- net PWAIT: now reaches P1.27 (RFU_1)
- net PWAIT: now also U41.12
- net PINTE: now reaches P1.28 (RFU_2)
- net PINTE: now also U41.4
- net A5: now reaches P1.29 (A5)
- net A5: now also U44.7 (O3a), U45.11, SW2.3 (C)
- net A4: now reaches P1.30 (A4)
- net A4: now also U43.3 (O1a), U45.3, SW2.6 (C)
- net A3: now reaches P1.31 (A3)
- net A3: now also U43.5 (O2a), U45.13, SW3.3 (C)
- net D1: now reaches P1.35 (DO1)
- net D1: now also U43.9 (O4a)
- net D0: now reaches P1.36 (DO0)
- net D0: now also U43.7 (O3a)
- net D4: now reaches P1.38 (DO4)
- net D4: now also U42.13 (O6b)
- net D5: now reaches P1.39 (DO5)
- net D5: now also U42.11 (O5b)
- net D6: now reaches P1.40 (DO6)
- net D6: now also U42.9 (O4a)
- net SMI: now reaches P1.44 (sM1)
- net SMI: now also U41.6
- net SOUT: now reaches P1.45 (sOUT)
- net SOUT: now also U34.4, U41.8
- net SINP: now reaches P1.46 (sINP)
- net SINP: now also U31.2, U34.11
- net SMEMR: now reaches P1.47 (sMEMR)
- net SMEMR: now also U31.12
- net SHLTA: now reaches P1.48 (sHLTA)
- net SHLTA: now also U31.10
- net MREQ: now reaches P1.65 (NDEF2)
- net MREQ: now also U44.3 (O1a)
- net RFSH: now reaches P1.66 (NDEF3)
- net RFSH: now also U44.13 (O6b)
- net PHOLD: now reaches P1.74 (HOLD*)
- net PHOLD: now also U34.2, U47.8
- net PRESET: now reaches P1.75 (RESET*)
- net PRESET: now also U26.10 (~{S})
- net PSYNC: now reaches P1.76 (pSYNC)
- net PSYNC: now also U41.2
- net PWR: now reaches P1.77 (pWR*)
- net PWR: now also U44.5 (O2a), U46.11
- net PDBIN: now reaches P1.78 (pDBIN)
- net PDBIN: now also U34.10, U41.10
- net A0: now reaches P1.79 (A0)
- net A0: now also U25.2, U44.11 (O5b), U46.9
- net A1: now reaches P1.80 (A1)
- net A1: now also U14.6, U44.9 (O4a), U46.5
- net A2: now reaches P1.81 (A2)
- net A2: now also U43.13 (O6b), U45.1, SW3.6 (C)
- net A6: now reaches P1.82 (A6)
- net A6: now also U43.11 (O5b), U45.5, SW1.6 (C)
- net A7: now reaches P1.83 (A7)
- net A7: now also U45.9, SW35.3 (C)
- net D2: now reaches P1.88 (DO2)
- net D2: now also U42.3 (O1a)
- net D3: now reaches P1.89 (DO3)
- net D3: now also U42.5 (O2a)
- net D7: now reaches P1.90 (DO7)
- net D7: now also U42.7 (O3a)
- net SINTA: now reaches P1.96 (sINTA)
- net SINTA: now also U31.4
- net SWO: now reaches P1.97 (sWO*)
- net SWO: now also U31.6
- net SSTACK: now reaches P1.98 (ERROR*)
- net SSTACK: now also U31.8
- net at U31.9: now also U26.2 (D), U31.1, U31.11, U31.13, U31.3, U31.5, U38.9 (Q), U41.1, U41.11, U41.13, U41.3, U41.5, U41.9
- net at U38.12 (D), U47.13, U47.3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: now also U47.11, U48.10, U48.11
- net at U22.10 (Q2): now also U43.10 (I4)
- net at U22.13 (E01): now also J11.13 (Pin_13), U13.1 (CP1..3), U22.4 (E23), U23.13 (E01), U23.4 (E23), U32.13 (E01), U32.4 (E23), U33.13 (E01), U33.4 (E23)
- net at U22.15 (Q1): now also U42.2 (I1)
- net at U22.16 (Q0): now also U42.4 (I2)
- net at U22.2 (D0): now also U21.6 (Q3)
- net at U22.3 (D1): now also U21.10 (Q4)
- net at U22.6 (D2): now also U21.11 (Q5)
- net at U22.7 (D3): now also U21.12 (Q6)
- net at U22.9 (Q3): now also U43.6 (I3)
- net at U36.12, U37.12: now also U27.5 (Q), U34.13
- net at U25.1: now also U15.1, U46.6
- net at U25.11: now also U14.12, U15.11, SW2.5 (B)
- net at U25.12: now also U14.11, U15.12, SW3.5 (B)
- net at U25.3: now also U14.4, U15.3, SW3.2 (B)
- net at U25.4: now also U14.3, U15.4, SW2.2 (B)
- net at U25.5: now also U14.2, U15.5, SW1.5 (B)
- net at U25.6: now also U14.1, U15.6, SW35.2 (B)
- net at U25.8: now also U24.12
- net at U16.3 (C), U27.3 (C), U37.5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: now also J11.12 (Pin_12), U48.1, U48.2, U48.6
- net at U24.1: now also J11.9 (Pin_9)
- net at U24.2: now also U14.8
- net at U24.3: now also U24.11, U24.5, U34.6
- net at U42.1 (OEa): now also J11.7 (Pin_7), U38.8 (~{Q}), U42.15 (OEb), U43.1 (OEa), U43.15 (OEb), U44.1 (OEa), U44.15 (OEb)
- net at U42.10 (I4): now also U32.15 (Q1)
- net at U42.12 (I5): now also U32.10 (Q2)
- net at U42.14 (I6): now also U32.9 (Q3)
- net at U42.6 (I3): now also U32.16 (Q0)
- net at U17.1 (~{R}), U17.13 (~{R}), U17.2 (D)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: now also U38.5 (Q), U47.9
- net at U13.11 (Q3): now also U12.14 (CP0), U23.3 (D1)
- net at U13.2 (R0(1)): now also J11.3 (Pin_3), U12.2 (R0(1)), U12.3 (R0(2)), U13.3 (R0(2))
- net at U13.8 (Q2): now also U23.7 (D3)
- net at J11.1 (Pin_1): now also U28.12, U28.13
- net at J11.10 (Pin_10): now also U24.13
- net at J11.11 (Pin_11): now also U24.4
- net at J11.14 (Pin_14): now also U32.2 (D0)
- net at J11.15 (Pin_15): now also U21.8 (CP)
- net at J11.2 (Pin_2): now also U12.11 (Q3), U33.7 (D3)
- net at J11.5 (Pin_5): now also U16.9 (Q)
- net at U45.4: now also SW2.4 (A)
- net at U45.2: now also SW3.4 (A)
- net at U15.2: now also U14.5, U46.8
- net at U15.8: now also U24.6, U24.9
- net at U46.10: now also U34.3
- net I5: now reaches U23.10 (Q2)
- net I5: now also U44.12 (I5)
- net at U23.15 (Q1): now also U43.14 (I6)
- net I4: now reaches U23.9 (Q3)
- net I4: now also U44.10 (I4)
- net at U34.5: now also U34.9, U48.12, U48.8
- net at U33.10 (Q2): now also U43.4 (I2)
- net at U33.15 (Q1): now also U43.2 (I1)
- net I3: now reaches U33.16 (Q0)
- net I3: now also U44.6 (I3)
- net at U33.2 (D0): now also U12.8 (Q2)
- net at U33.3 (D1): now also U12.9 (Q1)
- net at U33.6 (D2): now also U12.1 (CP1..3), U12.12 (Q0); no longer U12.9 (Q1)
- net at U33.9 (Q3): now also U43.12 (I5)
- net at U34.8: now also U24.8
- net at U45.8: now also SW35.1 (A)
- net at U45.6: now also SW1.4 (A)
- net at U45.12: now also SW3.1 (A)
- net at U32.3 (D1): now also U21.3 (Q0)
- net at U32.6 (D2): now also U21.4 (Q1)
- net at U32.7 (D3): now also U21.5 (Q2)
- net at U45.10: now also SW2.1 (A)
- net at U16.12 (D): now also U16.8 (~{Q})
- net at U21.1 (DSA): now also U21.2 (DSB), R2.2
- no-connect marks 0 -> 31
Other:
- moved on the sheet: U14A, U15A, U16B, U24A, U24D, U25A, U31A, U31B, U31C, U31D, U31E, U31F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

Commit message: Reproduction PCBs Final
Parts:
- R1: footprint footprints:R1206 -> Resistor_THT:R_Axial_DIN0204_L3.6mm_D1.6mm_P7.62mm_Horizontal
- R2: footprint footprints:R1206 -> Resistor_THT:R_Axial_DIN0204_L3.6mm_D1.6mm_P7.62mm_Horizontal; now not fitted; now left out of the parts list
- SW1: value SW_DPDT_x2 -> Port Select
- U14: footprint Package_DIP:DIP-10_W7.62mm -> Package_DIP:DIP-14_W7.62mm
- U15, U25: footprint (none) -> Package_DIP:DIP-14_W7.62mm
- renumbered SW35 to SW1, U1 to U36
Connections:
- net +5V: no longer R2.1
- net at J11.14 (Pin_14), U32.2 (D0): now also U21.1 (DSA), U21.2 (DSB)
- now unconnected: R2.2
Changed lines of the file:
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@@
 	)
 	(junction
+		(at 412.75 166.37)
+		(diameter 0)
+		(color 0 0 0 0)
+	)
+	(junction
 		(at 77.47 265.43)
 		(diameter 0)
@@
 	(wire
 		(pts
-			(xy 412.75 123.19) (xy 412.75 133.35)
-		)
-		(stroke
-			(width 0)
-			(type default)
-		)
-	)
-	(wire
-		(pts
 			(xy 133.35 334.01) (xy 133.35 350.52)
 		)
@@
 	(wire
 		(pts
-			(xy 382.27 166.37) (xy 466.09 166.37)
+			(xy 382.27 166.37) (xy 412.75 166.37)
 		)
 		(stroke
@@
 	(wire
 		(pts
+			(xy 412.75 166.37) (xy 466.09 166.37)
+		)
+		(stroke
+			(width 0)
+			(type default)
+		)
+	)
+	(wire
+		(pts
 			(xy 515.62 113.03) (xy 515.62 189.23)
 		)
@@
 	(wire
 		(pts
+			(xy 412.75 123.19) (xy 412.75 166.37)
+		)
+		(stroke
+			(width 0)
+			(type default)
+		)
+	)
+	(wire
+		(pts
 			(xy 524.51 151.13) (xy 524.51 123.19)
 		)
@@
 			)
 		)
-		(property "Footprint" ""
+		(property "Footprint" "Package_DIP:DIP-14_W7.62mm"
 			(at 161.29 384.81 0)
 			(effects
@@
 			)
 		)
-		(property "Value" "SW_DPDT_x2"
+		(property "Value" "Port Select"
 			(at 96.52 344.17 0)
 			(effects
@@
 		(dnp no)
 		(fields_autoplaced yes)
-		(property "Reference" "SW35"
+		(property "Reference" "SW1"
 			(at 96.52 332.74 0)
 			(effects
@@
 			(project ""
 				(path "/461ad1b3-df41-4c8f-89ba-1a25d4188f9a"
-					(reference "SW35")
+					(reference "SW1")
 					(unit 1)
 				)
@@
 			)
 		)
-		(property "Footprint" ""
+		(property "Footprint" "Package_DIP:DIP-14_W7.62mm"
 			(at 161.29 336.55 0)
 			(effects
@@
 			)
 		)
-		(property "Footprint" "Package_DIP:DIP-10_W7.62mm"
+		(property "Footprint" "Package_DIP:DIP-14_W7.62mm"
 			(at 30.48 36.83 0)
 			(effects
@@
 			)
 		)
-		(property "Footprint" "footprints:R1206"
+		(property "Footprint" "Resistor_THT:R_Axial_DIN0204_L3.6mm_D1.6mm_P7.62mm_Horizontal"
 			(at 275.844 175.006 90)
 			(effects
@@
 			)
 		)
-		(property "Footprint" ""
+		(property "Footprint" "Package_DIP:DIP-14_W7.62mm"
 			(at 52.07 36.83 0)
 			(effects
@@
 			)
 		)
-		(property "Footprint" ""
+		(property "Footprint" "Package_DIP:DIP-14_W7.62mm"
 			(at 73.66 36.83 0)
 			(effects
@@
 		(on_board yes)
 		(dnp no)
-		(property "Reference" "U1"
+		(property "Reference" "U36"
 			(at 284.7257 162.56 0)
 			(effects
@@
 			(project "88-CCC Board 2"
 				(path "/461ad1b3-df41-4c8f-89ba-1a25d4188f9a"
-					(reference "U1")
+					(reference "U36")
 					(unit 3)
 				)
@@
 	(symbol
 		(lib_id "power:+5V")
-		(at 412.75 140.97 0)
-		(mirror x)
-		(unit 1)
-		(exclude_from_sim no)
-		(in_bom yes)
-		(on_board yes)
-		(dnp no)
-		(property "Reference" "#PWR028"
-			(at 412.75 137.16 0)
-			(effects
-				(font
-					(size 1.27 1.27)
-				)
-				(hide yes)
-			)
-		)
-		(property "Value" "+5V"
-			(at 412.496 144.78 0)
-			(effects
-				(font
-					(size 1.27 1.27)
-				)
-			)
-		)
-		(property "Footprint" ""
-			(at 412.75 140.97 0)
-			(effects
-				(font
-					(size 1.27 1.27)
-				)
-				(hide yes)
-			)
-		)
-		(property "Datasheet" ""
-			(at 412.75 140.97 0)
-			(effects
-				(font
-					(size 1.27 1.27)
-				)
-				(hide yes)
-			)
-		)
-		(property "Description" "Power symbol creates a global label with name \"+5V\""
-			(at 412.75 140.97 0)
-			(effects
-				(font
-					(size 1.27 1.27)
-				)
-				(hide yes)
-			)
-		)
-		(pin "1"
-		)
-		(instances
-			(project "88-CCC Board 2"
-				(path "/461ad1b3-df41-4c8f-89ba-1a25d4188f9a"
-					(reference "#PWR028")
-					(unit 1)
-				)
-			)
-		)
-	)
-	(symbol
-		(lib_id "power:+5V")
 		(at 242.57 195.58 0)
 		(unit 1)
@@
 	(symbol
 		(lib_id "Device:R_US")
-		(at 412.75 137.16 0)
+		(at 410.21 160.02 0)
 		(mirror x)
 		(unit 1)
 		(exclude_from_sim no)
-		(in_bom yes)
-		(on_board yes)
-		(dnp no)
+		(in_bom no)
+		(on_board no)
+		(dnp yes)
 		(property "Reference" "R2"
-			(at 407.162 136.144 0)
+			(at 404.622 159.004 0)
 			(effects
 				(font
@@
 		)
 		(property "Value" "560"
-			(at 407.416 139.7 0)
+			(at 404.876 162.56 0)
 			(effects
 				(font
@@
 			)
 		)
-		(property "Footprint" "footprints:R1206"
-			(at 413.766 136.906 90)
+		(property "Footprint" "Resistor_THT:R_Axial_DIN0204_L3.6mm_D1.6mm_P7.62mm_Horizontal"
+			(at 411.226 159.766 90)
 			(effects
 				(font
@@
 		)
 		(property "Datasheet" "https://lcsc.com/product-detail/Chip-Resistor-Surface-Mount-UniOhm_1KR-102-5_C1469.html"
-			(at 412.75 137.16 0)
+			(at 410.21 160.02 0)
 			(effects
 				(font
@@
 		)
 		(property "Description" "Resistor, US symbol"
-			(at 412.75 137.16 0)
+			(at 410.21 160.02 0)
 			(effects
 				(font
@@
 		)
 		(property "MANUFACTURER" ""
-			(at 412.75 137.16 0)
+			(at 410.21 160.02 0)
 			(effects
 				(font
@@
 		)
 		(property "MAXIMUM_PACKAGE_HEIGHT" ""
-			(at 412.75 137.16 0)
+			(at 410.21 160.02 0)
 			(effects
 				(font
@@
 		)
 		(property "PARTREV" ""
-			(at 412.75 137.16 0)
+			(at 410.21 160.02 0)
 			(effects
 				(font
@@
 		)
 		(property "STANDARD" ""
-			(at 412.75 137.16 0)
+			(at 410.21 160.02 0)
 			(effects
 				(font
@@
 		)
 		(property "LCSC Part" "C1469"
-			(at 412.75 137.16 0)
+			(at 410.21 160.02 0)
 			(effects
 				(font
@@
 		)
 		(property "Sim.Device" ""
-			(at 412.75 137.16 0)
+			(at 410.21 160.02 0)
 			(effects
 				(font
@@
 		)
 		(property "Sim.Pins" ""
-			(at 412.75 137.16 0)
+			(at 410.21 160.02 0)
 			(effects
 				(font
@@
 		)
 		(property "Field5" ""
-			(at 412.75 137.16 0)
+			(at 410.21 160.02 0)
 			(effects
 				(font
@@
 		)
 		(property "LCSC" ""
-			(at 412.75 137.16 90)
+			(at 410.21 160.02 90)
 			(effects
 				(font
@@
 			)
 		)
-		(property "Footprint" "Package_DIP:DIP-10_W7.62mm"
+		(property "Footprint" "Package_DIP:DIP-14_W7.62mm"
 			(at 161.29 412.75 0)
 			(effects
