File: PCB/88-CCC Board 2/88-CCC Board 2.kicad_pcb (KiCad board)
At the start: 6 copper layers, 254 x 134.6 mm, 1 part, among them P1 S100_MALE

Commit message: Reproduction PCBs Final
Parts:
- added C10: 47uF, Capacitor_THT:C_Axial_L17.0mm_D7.0mm_P25.00mm_Horizontal, F.Cu at (23.2, 85.4)
- added C11: 47uF, Capacitor_THT:C_Axial_L17.0mm_D7.0mm_P25.00mm_Horizontal, F.Cu at (23.5, 124.2)
- added C2: 0.1uF, Capacitor_THT:C_Disc_D7.5mm_W5.0mm_P7.50mm, F.Cu at (30.1, 136.0)
- added C3: 0.1uF, Capacitor_THT:C_Disc_D7.5mm_W5.0mm_P7.50mm, F.Cu at (24.6, 89.2)
- added C4: 0.1uF, Capacitor_THT:C_Disc_D7.5mm_W5.0mm_P5.00mm, F.Cu at (50.7, 69.4)
- added C5: 0.1uF, Capacitor_THT:C_Disc_D7.5mm_W5.0mm_P5.00mm, F.Cu at (77.8, 43.7)
- added C6: 0.1uF, Capacitor_THT:C_Disc_D7.5mm_W5.0mm_P7.50mm, F.Cu at (253.8, 122.0)
- added C7: 0.1uF, Capacitor_THT:C_Disc_D7.5mm_W5.0mm_P7.50mm, F.Cu at (253.8, 96.0)
- added C8: 0.1uF, Capacitor_THT:C_Disc_D7.5mm_W5.0mm_P7.50mm, F.Cu at (253.8, 70.8)
- added C9: 0.1uF, Capacitor_THT:C_Disc_D7.5mm_W5.0mm_P7.50mm, F.Cu at (253.8, 45.1)
- added J11: To Board 1, Package_DIP:DIP-16_W7.62mm, F.Cu at (228.7, 50.1)
- added R1: 1K, Resistor_THT:R_Axial_DIN0204_L3.6mm_D1.6mm_P7.62mm_Horizontal, F.Cu at (106.1, 45.2)
- added SW1: Port Select, Package_DIP:DIP-6_W7.62mm, F.Cu at (109.7, 101.0)
- added SW2: SW_DPDT_x2, Package_DIP:DIP-6_W7.62mm, F.Cu at (118.0, 101.0)
- added SW3: SW_DPDT_x2, Package_DIP:DIP-6_W7.62mm, F.Cu at (126.2, 101.0)
- added U12: 7493, Package_DIP:DIP-14_W7.62mm, F.Cu at (198.6, 50.1)
- added U13: 7493, Package_DIP:DIP-14_W7.62mm, F.Cu at (170.0, 50.1)
- added U14: 7430, Package_DIP:DIP-14_W7.62mm, F.Cu at (142.5, 50.1)
- added U15: 7430, Package_DIP:DIP-14_W7.62mm, F.Cu at (112.4, 50.1)
- added U16: 7474, Package_DIP:DIP-14_W7.62mm, F.Cu at (84.8, 50.1)
- added U17: 7474, Package_DIP:DIP-14_W7.62mm, F.Cu at (55.9, 50.1)
- added U18: L7805, Package_TO_SOT_THT:TO-220-3_Horizontal_TabDown, F.Cu at (27.6, 60.3)
- added U21: 74HC164, Package_DIP:DIP-14_W7.62mm, F.Cu at (230.0, 76.0)
- added U22: 7475, Package_DIP:DIP-16_W7.62mm, F.Cu at (200.0, 76.0)
- added U23: 7475, Package_DIP:DIP-16_W7.62mm, F.Cu at (170.0, 76.0)
- added U24: 7402, Package_DIP:DIP-14_W7.62mm, F.Cu at (141.2, 76.0)
- added U25: 7430, Package_DIP:DIP-14_W7.62mm, F.Cu at (112.4, 76.0)
- added U26: 7474, Package_DIP:DIP-14_W7.62mm, F.Cu at (83.6, 76.0)
- added U27: 7474, Package_DIP:DIP-14_W7.62mm, F.Cu at (57.3, 76.0)
- added U28: 7400, Package_DIP:DIP-14_W7.62mm, F.Cu at (29.8, 76.0)
- added U31: 7405, Package_DIP:DIP-14_W7.62mm, F.Cu at (230.0, 101.0)
- added U32: 7475, Package_DIP:DIP-16_W7.62mm, F.Cu at (198.7, 101.0)
- added U33: 7475, Package_DIP:DIP-16_W7.62mm, F.Cu at (168.7, 101.0)
- added U34: 7410, Package_DIP:DIP-14_W7.62mm, F.Cu at (141.2, 101.0)
- added U36: 7402, Package_DIP:DIP-14_W7.62mm, F.Cu at (83.6, 101.0)
- added U37: 7400, Package_DIP:DIP-14_W7.62mm, F.Cu at (57.3, 101.0)
- added U38: 7474, Package_DIP:DIP-14_W7.62mm, F.Cu at (28.6, 101.0)
- added U41: 7405, Package_DIP:DIP-14_W7.62mm, F.Cu at (228.6, 127.0)
- added U42: 74367, Package_DIP:DIP-16_W7.62mm, F.Cu at (199.8, 127.0)
- added U43: 74367, Package_DIP:DIP-16_W7.62mm, F.Cu at (169.9, 127.0)
- added U44: 74367, Package_DIP:DIP-16_W7.62mm, F.Cu at (141.0, 127.0)
- added U45: 7404, Package_DIP:DIP-14_W7.62mm, F.Cu at (112.3, 127.0)
- added U46: 7404, Package_DIP:DIP-14_W7.62mm, F.Cu at (84.8, 127.0)
- added U47: 7405, Package_DIP:DIP-14_W7.62mm, F.Cu at (57.4, 127.0)
- added U48: 7400, Package_DIP:DIP-14_W7.62mm, F.Cu at (29.6, 127.0)
Connections:
- net Net-(J5-Pin_2) renamed -16V
- P1 pad 1: Net-(J5-Pin_1) -> +8V
- P1 pad 18: unconnected-(P1-SDSB*-Pad18) -> SDSB
- P1 pad 19: unconnected-(P1-CDSB*-Pad19) -> CDSB
- P1 pad 2: unconnected-(P1-+16_V-Pad2) -> +16V
- P1 pad 22: unconnected-(P1-ADSB*-Pad22) -> ADSB
- P1 pad 23: unconnected-(P1-DODSB*-Pad23) -> DODSB
- P1 pad 24: unconnected-(P1-PHI-Pad24) -> 02
- P1 pad 26: unconnected-(P1-pHDLA-Pad26) -> PHLDA
- P1 pad 27: unconnected-(P1-RFU_1-Pad27) -> PWAIT
- P1 pad 28: unconnected-(P1-RFU_2-Pad28) -> PINTE
- P1 pad 29: unconnected-(P1-A5-Pad29) -> A5
- P1 pad 30: unconnected-(P1-A4-Pad30) -> A4
- P1 pad 31: unconnected-(P1-A3-Pad31) -> A3
- P1 pad 35: unconnected-(P1-DO1-Pad35) -> D1
- P1 pad 36: unconnected-(P1-DO0-Pad36) -> D0
- P1 pad 38: unconnected-(P1-DO4-Pad38) -> D4
- P1 pad 39: unconnected-(P1-DO5-Pad39) -> D5
- P1 pad 40: unconnected-(P1-DO6-Pad40) -> D6
- P1 pad 44: unconnected-(P1-sM1-Pad44) -> SMI
- P1 pad 45: unconnected-(P1-sOUT-Pad45) -> SOUT
- P1 pad 46: unconnected-(P1-sINP-Pad46) -> SINP
- P1 pad 47: unconnected-(P1-sMEMR-Pad47) -> SMEMR
- P1 pad 48: unconnected-(P1-sHLTA-Pad48) -> SHLTA
- P1 pad 49: unconnected-(P1-CLOCK-Pad49) -> CLOCK
- P1 pad 51: unconnected-(P1-+8_V-Pad51) -> +8V
- P1 pad 65: unconnected-(P1-NDEF2-Pad65) -> MREQ
- P1 pad 66: unconnected-(P1-NDEF3-Pad66) -> RFSH
- P1 pad 74: unconnected-(P1-HOLD*-Pad74) -> PHOLD
- P1 pad 75: /S100_RESET_P75 -> PRESET
- P1 pad 76: unconnected-(P1-pSYNC-Pad76) -> PSYNC
- P1 pad 77: unconnected-(P1-pWR*-Pad77) -> PWR
- P1 pad 78: unconnected-(P1-pDBIN-Pad78) -> PDBIN
- P1 pad 79: unconnected-(P1-A0-Pad79) -> A0
- P1 pad 80: unconnected-(P1-A1-Pad80) -> A1
- P1 pad 81: unconnected-(P1-A2-Pad81) -> A2
- P1 pad 82: unconnected-(P1-A6-Pad82) -> A6
- P1 pad 83: unconnected-(P1-A7-Pad83) -> A7
- P1 pad 88: unconnected-(P1-DO2-Pad88) -> D2
- P1 pad 89: unconnected-(P1-DO3-Pad89) -> D3
- P1 pad 90: unconnected-(P1-DO7-Pad90) -> D7
- P1 pad 96: unconnected-(P1-sINTA-Pad96) -> SINTA
- P1 pad 97: unconnected-(P1-sWO*-Pad97) -> SWO
- P1 pad 98: unconnected-(P1-ERROR*-Pad98) -> SSTACK
Routing:
- net +5V: track 0.00 -> 1208.5 mm, vias 0 -> 6
- net GND: track 0.00 -> 1193.6 mm, vias 0 -> 9
- net Net-(J11-Pin_7): track 0.00 -> 354.8 mm, vias 0 -> 4
- net Net-(J11-Pin_12): track 0.00 -> 344.9 mm, vias 0 -> 4
- net Net-(U26A-D): track 0.00 -> 296.9 mm, vias 0 -> 1
- net Net-(J11-Pin_1): track 0.00 -> 204.0 mm, vias 0 -> 1
- net Net-(U17A-C): track 0.00 -> 183.3 mm, vias 0 -> 2
- net A1: track 0.00 -> 180.0 mm, vias 0 -> 6
- net Net-(J11-Pin_13): track 0.00 -> 166.5 mm, vias 0 -> 1
- net PDBIN: track 0.00 -> 166.0 mm, vias 0 -> 6
- net Net-(U34-Pad5): track 0.00 -> 164.0 mm, vias 0 -> 2
- net A2: track 0.00 -> 163.3 mm, vias 0 -> 2
- net SOUT: track 0.00 -> 161.8 mm, vias 0 -> 2
- net A0: track 0.00 -> 158.6 mm, vias 0 -> 6
- net A4: track 0.00 -> 158.4 mm, vias 0 -> 5
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Other:
- copper layers 6 -> 2
- board text added: "1"
- board text added: "1K"
- board text added: "2"
- board text added: "3"
- board text added: "4"
- board text added: "7400"
- board text added: "7402"
- board text added: "7404"
- board text added: "7405"
- board text added: "7410"
- board text added: "74134"
- board text added: "7430"
- board text added: "74367"
- board text added: "7474"
- board text added: "7475"
- board text added: "7493"
- board text added: "8 7 6 5 4 3 2 1"
- board text added: "CROMEMCO 88 CCC BOARD 2"
- board text added: "PORT SELECT"
- board text added: "REPRODUCTION 2026 ARON HOEKSTRA"
- board text added: "TO BOARD 1"

Commit message: Reproduction PCBs Final
Routing:
- net GND: vias 9 -> 8
Changed lines of the file:
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@@
-		(net 1)
-	)
-	(via
-		(at 46.1 47.15)
-		(size 0.9)
-		(drill 0.4)
-		(layers "F.Cu" "B.Cu")
 		(net 1)
 	)
